Commit message: Improved rover URDF
Added backup of previous version of URDF that was submitted for report 2.

File: description/rover_backup.xacro.urdf (robot description, URDF)
Before this commit: robot car, 5 links, 4 joints
Links:
- removed link left_wheel_link
- removed link right_wheel_link
- added link wheel_bl_link; collision cylinder length=${wheel_width} radius=${wheel_diameter}; visual cylinder length=${wheel_width} radius=${wheel_diameter}
- added link wheel_br_link; collision cylinder length=${wheel_width} radius=${wheel_diameter}; visual cylinder length=${wheel_width} radius=${wheel_diameter}
Joints:
- removed joint left_wheel_joint
- removed joint right_wheel_joint
- added joint wheel_bl_joint: type continuous, parent chasis_link, child wheel_bl_link, origin xyz=${-(chasis_x/2 + wheel_width/2)} ${-(chasis_x - wheel_width/2)} ${chasis_z/2} rpy=0 ${-pi/2} 0, axis 0 0 1
- added joint wheel_br_joint: type continuous, parent chasis_link, child wheel_br_link, origin xyz=${chasis_x/2 + wheel_width/2} ${-(chasis_x - wheel_width/2)} ${chasis_z/2} rpy=0 ${pi/2} 0, axis 0 0 -1
- joint wheel_front_joint: origin xyz=0.16 0 ${-front_wheel_diameter} -> xyz=0 ${chasis_y/3} 0
