Commit message: updated many files.
Updated Gazebo file to enable materials in gazebo.
Added Gazebo control file.
updated gazebo file to match new joint and link names.

File: description/autonomous_rover.urdf.xacro (robot description, xacro)
@@ -2,3 +2,4 @@
 <robot xmlns:xacro="http://www.ros.org/wiki/xacro" name="rover">
     <xacro:include filename="rover.xacro"/>
+    <xacro:include filename="gazebo_control.xacro"/>
 </robot>

File: description/example_gazebo.xacro (robot description, xacro)
@@ -4,10 +4,10 @@
     <!-- Instead, we need to add gazebo tags for our links that refer to Gazebo materials -->
     <gazebo reference="chasis_link">
-        <material>Gazebo/Grey</material>
+        <material>Gazebo/Yellow</material>
     </gazebo>
-    <gazebo reference="wheel_br_link">
+    <gazebo reference="right_wheel_link">
         <material>Gazebo/Orange</material>
     </gazebo>
-    <gazebo reference="wheel_bl_link">
+    <gazebo reference="left_wheel_link">
         <material>Gazebo/Orange</material>
     </gazebo>
@@ -19,6 +19,6 @@
             filename="libgazebo_ros_joint_state_publisher.so">
             <update_rate>20</update_rate>
-            <joint_name>wheel_br_joint</joint_name>
-            <joint_name>wheel_bl_joint</joint_name>
+            <joint_name>right_wheel_joint</joint_name>
+            <joint_name>left_wheel_joint</joint_name>
         </plugin>
     </gazebo>

File: description/rover.xacro (robot description, xacro)
@@ -114,3 +114,4 @@
         </xacro:inertial_sphere>
     </link>
+    <xacro:include filename="example_gazebo.xacro" />
 </robot>

Commit message: Added LiDAR files for simulation
Publishes ray scans to laser scan topic.

File: description/autonomous_rover.urdf.xacro (robot description, xacro)
@@ -3,3 +3,4 @@
     <xacro:include filename="rover.xacro"/>
     <xacro:include filename="gazebo_control.xacro"/>
+    <xacro:include filename="lidar.xacro"/>
 </robot>

File: description/general_include.xacro (robot description, xacro)
@@ -10,4 +10,7 @@
     <material name="blue">
         <color rgba="0.2 0.2 1 1"/>
+    </material>
+    <material name="red">
+        <color rgba=" 0.8 0.1 0.1 1"/>
     </material>
     <!-- Specify some standard inertial calculations https://en.wikipedia.org/wiki/List_of_moments_of_inertia -->

Commit message: Added ros2 control files
YAML file in config folder sets up the control parameters.

File: description/autonomous_rover.urdf.xacro (robot description, xacro)
@@ -1,6 +1,7 @@
 <?xml version="1.0"?>
 <robot xmlns:xacro="http://www.ros.org/wiki/xacro" name="rover">
+    <xacro:include filename="ros2_control.xacro"/>
     <xacro:include filename="rover.xacro"/>
-    <xacro:include filename="gazebo_control.xacro"/>
+    <!-- <xacro:include filename="gazebo_control.xacro"/> -->
     <xacro:include filename="lidar.xacro"/>
 </robot>

File: description/lidar.xacro (robot description, xacro)
@@ -24,30 +24,32 @@
     </link>
     <gazebo reference="lidar_frame">
+        <material>Gazebo/Red</material>
         <sensor name="lidar" type="ray">
-        <pose> 0 0 0 0 0 0 </pose>
-        <visualize> true </visualize>
-        <update_rate>10</update_rate>
-        <ray>
-            <scan>
-                <horizontal>
-                    <samples> 360 </samples>
-                    <resolution> 1 </resolution>
-                    <min_angle>-3.14</min_angle>
-                    <max_angle>3.14</max_angle>
-                </horizontal>
-            </scan>
-            <range>
-                <min>0.3</min>
-                <max>12</max>
-                <resolution> 1</resolution>
-            </range>
-        </ray>
-        <plugin name="lidar_controller" filename="libgazebo_ros_ray_sensor.so">
-            <ros>
-                <argument> ~/out:=scan </argument>
-            </ros>
-            <output_type>s ensor_msgs/LaserScan </output_type>
-            <frame_name> lidar_frame </frame_name>
-        </plugin>
-    </sensor>
+            <pose> 0 0 0 0 0 0 </pose>
+            <visualize> true </visualize>
+            <update_rate>10</update_rate>
+            <ray>
+                <scan>
+                    <horizontal>
+                        <samples> 360 </samples>
+                        <resolution> 1 </resolution>
+                        <min_angle>-3.14</min_angle>
+                        <max_angle>3.14</max_angle>
+                    </horizontal>
+                </scan>
+                <range>
+                    <min>0.3</min>
+                    <max>12</max>
+                    <resolution> 1</resolution>
+                </range>
+            </ray>
+            <plugin name="laser_controller" filename="libgazebo_ros_ray_sensor.so">
+                <ros>
+                    <argument> ~/out:=scan </argument>
+                </ros>
+                <output_type> sensor_msgs/LaserScan </output_type>
+                <frame_name> lidar_frame </frame_name>
+            </plugin>
+        </sensor>
+    </gazebo>
 </robot>
